File: PowerBoard.kicad_pcb (KiCad board)
At the start: 2 copper layers, 100 x 90 mm, 29 parts, among them J1 Main Pack, J2 Supp bat, J3 Main Connection, J4 Main Connection, J5 12v, J6 12vM, J7 12vS, Q1 IRLR7843TRPBF, Q2 IRLR7843TRPBF, U1 CN-A110, U2 LTC4357MS8, U3 LTC4357MS8

Commit message: Adding automation
Parts:
- moved J1 1.60 mm to (62.1, 67.0)
- moved J2 0.15 mm to (62.1, 48.0)
- moved J6 0.12 mm to (157.9, 54.9)
- moved J5 0.05 mm to (157.8, 108.7)
Routing:
- net /12vS: track 18.8 -> 16.1 mm
- net -BATT: track 24.9 -> 25.6 mm
Other:
- board text added: "Power Board Ideal Diode Version 2.0.0 John Carr Solar Gators"
- board text removed: "Power Board Ideal Diode Version 0.1.0 John Carr Solar Gators"
