File: PowerBoard.kicad_sch (KiCad schematic)
At the start: 29 parts, among them J1 Main Pack, J2 Supp bat, J3 Main Connection, J4 Main Connection, J5 12v, J6 12vM, J7 12vS, Q1 IRLR7843TRPBF, Q2 IRLR7843TRPBF, U1 CN-A110, U2 LTC4357MS8, U3 LTC4357MS8

Commit message: Fix for automation
Parts:
- C1: LCSC Part C28323 -> (none); LCSC# (none) -> C28323
- C3, C4: LCSC Part C14663 -> (none); LCSC# (none) -> C14663
- D1: LCSC Part C64898 -> (none); LCSC# (none) -> C64898
- Q1, Q2: LCSC Part C21988 -> (none); LCSC# (none) -> C21988
- R1, R2: LCSC Part C22775 -> (none); LCSC# (none) -> C22775
Changed lines of the file:
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@@
       (effects (font (size 1.27 1.27)) hide)
     )
-    (property "LCSC Part" "C64898" (id 4) (at 52.07 27.94 90)
+    (property "LCSC#" "C64898" (id 4) (at 52.07 27.94 90)
       (effects (font (size 1.27 1.27)) hide)
     )
@@
       (effects (font (size 1.27 1.27)) hide)
     )
-    (property "LCSC Part" "C28323" (id 4) (at 102.87 26.67 0)
+    (property "LCSC#" "C28323" (id 4) (at 102.87 26.67 0)
       (effects (font (size 1.27 1.27)) hide)
     )
@@
       (effects (font (size 1.27 1.27)) hide)
     )
-    (property "LCSC Part" "C21988" (id 4) (at 76.2 91.44 90)
+    (property "LCSC#" "C21988" (id 4) (at 76.2 91.44 90)
       (effects (font (size 1.27 1.27)) hide)
     )
@@
       (effects (font (size 1.27 1.27)) hide)
     )
-    (property "LCSC Part" "C21988" (id 4) (at 76.2 142.24 90)
+    (property "LCSC#" "C21988" (id 4) (at 76.2 142.24 90)
       (effects (font (size 1.27 1.27)) hide)
     )
@@
       (effects (font (size 1.27 1.27)) hide)
     )
-    (property "LCSC Part" "C22775" (id 4) (at 88.9 102.87 0)
+    (property "LCSC#" "C22775" (id 4) (at 88.9 102.87 0)
       (effects (font (size 1.27 1.27)) hide)
     )
@@
       (effects (font (size 1.27 1.27)) hide)
     )
-    (property "LCSC Part" "C14663" (id 4) (at 88.9 110.49 0)
+    (property "LCSC#" "C14663" (id 4) (at 88.9 110.49 0)
       (effects (font (size 1.27 1.27)) hide)
     )
@@
       (effects (font (size 1.27 1.27)) hide)
     )
-    (property "LCSC Part" "C22775" (id 4) (at 88.9 153.67 0)
+    (property "LCSC#" "C22775" (id 4) (at 88.9 153.67 0)
       (effects (font (size 1.27 1.27)) hide)
     )
@@
       (effects (font (size 1.27 1.27)) hide)
     )
-    (property "LCSC Part" "C14663" (id 4) (at 88.9 161.29 0)
-      (effects (font (size 1.27 1.27)) hide)
-    )
+    (property "LCSC#" "C14663" (id 4) (at 88.9 161.29 0)
+      (effects (font (size 1.27 1.27)) hide)
+    )
